File: AudioAmp.kicad_pcb (KiCad board)
At the start: 4 copper layers, 97 parts, among them J101 Power Terminal, J102 USB C Port, J103 Mic 1 Connector, J104 Mic 2 Connector, J105 GPIO 0 Connector, J106 GPIO 1 Connector, J107 GPIO 2 Connector, J108 GPIO 3 Connector, J109 Speaker Right Connector, J110 Speaker Left Connector, U201 STM32F446RCTx, U401 TLV75733PDRV, Y201 Crystal_GND24

Commit message: ara ara
Parts:
- removed R401, R402: 2.2k, Resistor_SMD:R_0402_1005Metric_Pad0.72x0.64mm_HandSolder
- added C513: 0.1u, Capacitor_SMD:C_0603_1608Metric_Pad1.08x0.95mm_HandSolder, F.Cu at (105.5, 38.4)
- added C514: 0.1u, Capacitor_SMD:C_0603_1608Metric_Pad1.08x0.95mm_HandSolder, F.Cu at (81.0, 41.0)
- added J501: SWD Connector, Connector_PinSocket_1.00mm:PinSocket_1x04_P1.00mm_Vertical, F.Cu at (-72.2, 67.2)
- added R513: 2.2k, Resistor_SMD:R_0402_1005Metric_Pad0.72x0.64mm_HandSolder, F.Cu at (117.6, 36.5)
- added R514: 2.2k, Resistor_SMD:R_0402_1005Metric_Pad0.72x0.64mm_HandSolder, F.Cu at (116.4, 37.5)
- added R515: 2.2k, Resistor_SMD:R_0402_1005Metric_Pad0.72x0.64mm_HandSolder, F.Cu at (103.5, 35.9)
- added R516: 2.2k, Resistor_SMD:R_0402_1005Metric_Pad0.72x0.64mm_HandSolder, F.Cu at (102.4, 34.9)
- added U503: ~, Diode_SMD:D_SOD-923, F.Cu at (-67.4, 50.5)
- added U504: ~, Diode_SMD:D_SOD-923, F.Cu at (-67.4, 52.5)
- added U505: ~, Diode_SMD:D_SOD-923, F.Cu at (-67.4, 54.5)
- C204, C205, C301, C303, C304, C307, C501, C502, C503, C504, C505, C506, C507, C508, C509, C511, C512, R501, R502, R503, R504, R506, R507, R508, R509, R510, R511, R512, U104, U105, U114, U115, U116, U117, U501, U502: moved to F.Cu
- R207, R208: footprint Resistor_SMD:R_0603_1608Metric_Pad0.98x0.95mm_HandSolder -> Resistor_SMD:R_0402_1005Metric_Pad0.72x0.64mm_HandSolder
- R302, R303: footprint Resistor_SMD:R_0612_1632Metric_Pad1.18x3.40mm_HandSolder -> Resistor_SMD:R_0402_1005Metric_Pad0.72x0.64mm_HandSolder
- moved U109 170.5 mm to (-70.1, 44.7)
- moved U111 169.8 mm to (-70.1, 48.6)
- moved U106 164.8 mm to (-72.8, 50.5)
- moved U110 159.9 mm to (-70.1, 46.6)
- moved J105 158.6 mm to (-72.5, 40.2)
- moved J106 158.6 mm to (-69.2, 40.2)
- moved J107 158.6 mm to (-65.8, 40.2)
- moved J108 158.6 mm to (-62.5, 40.2)
- moved U113 157.5 mm to (-70.1, 52.5)
- moved U107 157.3 mm to (-72.8, 52.5)
- moved U108 153.1 mm to (-72.8, 54.5)
- moved U112 146.6 mm to (-70.1, 50.5)
- moved U103 133.9 mm to (-72.8, 44.7)
- moved U101 130.5 mm to (-73.1, 72.9)
- moved J101 127.2 mm to (-84.5, 41.8), turned to 0 degrees
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Connections:
- net Net-(U201-PA4) renamed /MCU/i2s_ws _series
- net Net-(U201-PA5) renamed /MCU/i2s_clk_series
- net Net-(U201-PA7) renamed /MCU/i2s_1_sd_sereis
- net Net-(U201-PC4) renamed /MCU/i2s_mclk_series
- net Net-(U301-SDOUT(M/~{S})) renamed /Codec/codec_sdout_sereis
- C501 pad 1: Net-(U501C-+) -> Net-(U501C--)
- C502 pad 1: Net-(U501D-+) -> Net-(U501D--)
- C508 pad 1: Net-(U501B-+) -> Net-(U501B--)
- J103 pad 2: GNDS -> GND
- J104 pad 2: GNDS -> GND
- J109 pad 1: SPKR_RIGHT_P_BUF -> GND
- J109 pad 3: GNDS -> SPKR_RIGHT_P_BUF
- J110 pad 1: SPKR_LEFT_P_BUF -> GND
- J110 pad 3: GNDS -> SPKR_LEFT_P_BUF
- U104 pad 2: GNDS -> GND
- U105 pad 2: GNDS -> GND
- U114 pad 2: GNDS -> GND
- U115 pad 2: GNDS -> GND
- U116 pad 2: GNDS -> GND
- U117 pad 2: GNDS -> GND
- U201 pad 26: unconnected-(U201-PB0-Pad26) -> I2S_2_SD
- U201 pad 29: I2S_CLK -> unconnected-(U201-PB10-Pad29)
- U201 pad 33: I2S_WS -> unconnected-(U201-PB12-Pad33)
- U201 pad 50: unconnected-(U201-PA15-Pad50) -> I2S_CLK
- U201 pad 51: unconnected-(U201-PC10-Pad51) -> I2S_CLK
- U201 pad 9: I2S_2_SD -> unconnected-(U201-PC1-Pad9)
- U301 pad 24: SPKR_RIGHT_N -> SPKR_LEFT_N
- U301 pad 25: SPKR_RIGHT_P -> SPKR_LEFT_P
- U301 pad 26: SPKR_LEFT_P -> SPKR_RIGHT_N
- U301 pad 27: SPKR_LEFT_N -> SPKR_RIGHT_P
- U501 pad 10: Net-(U501C-+) -> SPKR_LEFT_P
- U501 pad 12: Net-(U501D-+) -> SPKR_LEFT_N
- U501 pad 13: SPKR_LEFT_N -> Net-(U501D--)
- U501 pad 14: Net-(U501D-+) -> Net-(U501D--)
- U501 pad 5: Net-(U501B-+) -> SPKR_RIGHT_N
- U501 pad 6: SPKR_RIGHT_N -> Net-(U501B--)
- U501 pad 7: Net-(U501B-+) -> Net-(U501B--)
- U501 pad 8: Net-(U501C-+) -> Net-(U501C--)
- U501 pad 9: SPKR_LEFT_P -> Net-(U501C--)
Routing:
- net +3V3: track 92.5 -> 1.72 mm, vias 6 -> 0
- net +5V: track 86.5 -> 19.1 mm, vias 2 -> 5
- net I2S_CLK: track 42.5 -> 0.00 mm, vias 2 -> 0
- net I2S_1_SD: track 35.4 -> 0.00 mm, vias 2 -> 0
- net I2S_MCLK: track 33.4 -> 0.00 mm
- net I2C_1_SCL: track 29.1 -> 0.00 mm, vias 2 -> 0
- net I2C_1_SDA: track 29.0 -> 0.00 mm, vias 2 -> 0
- net CODEC_RST: track 26.9 -> 0.00 mm
- net I2S_WS: track 26.3 -> 0.00 mm, vias 2 -> 0
- net GND: track 72.1 -> 51.3 mm, vias 26 -> 25
- net GNDS: track 19.6 -> 4.66 mm, vias 7 -> 0
- net /MCU/crystal_A: track 14.0 -> 0.00 mm
- net MIC_2_IN_BUF: track 25.4 -> 12.6 mm, vias 1 -> 0
- net SPKR_LEFT_N: track 21.9 -> 9.55 mm, vias 1 -> 0
- net SPKR_LEFT_P: track 18.6 -> 7.55 mm, vias 1 -> 0
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- removed copper zone on F.Cu, net /Connectors/5V_INPUT
- removed copper zone on In1.Cu, net GND
