File: MCU.kicad_sch (KiCad schematic)
At the start: 20 parts, among them U1 STM32F446RCTx, Y201 Crystal_GND24

Commit message: ara ara
Parts:
- R1: footprint Resistor_SMD:R_0603_1608Metric_Pad0.98x0.95mm_HandSolder -> Resistor_SMD:R_0402_1005Metric_Pad0.72x0.64mm_HandSolder
Connections:
- net I2S_2_SD: now also U1.26 (PB0); no longer U1.9 (PC1)
- net I2S_CLK: now also U1.50 (PA15), U1.51 (PC10); no longer U1.29 (PB10)
- net I2S_WS: no longer U1.33 (PB12)
- net i2s_clk_series: now reaches R1.1, U1.21 (PA5)
- net i2s_ws _series: now reaches R1.1, U1.20 (PA4)
- net i2s_1_sd_sereis: now reaches R1.1, U1.23 (PA7)
- net i2s_mclk_series: now reaches R1.2, U1.24 (PC4)
Other:
- moved on the sheet: R1
