File: analog.kicad_sch (KiCad schematic)
At the start: 26 parts

Commit message: ara ara
Parts:
- added C1 (x2): 0.1u, Capacitor_SMD:C_0603_1608Metric_Pad1.08x0.95mm_HandSolder, symbol Device:C
- added R401 (x2), R402 (x2): 2.2k, Resistor_SMD:R_0402_1005Metric_Pad0.72x0.64mm_HandSolder, symbol Device:R_US
Connections:
- net +5V: now also C1.1, C1.2, R401.1, R401.1
- net GND: now also C1.1, C1.2, R402.2, R402.2
- net GNDS: now also R401.2, R401.2, R402.1, R402.1
- net SPKR_LEFT_N: now also U501.12 (+); no longer U501.13 (-)
- net SPKR_LEFT_P: now also U501.10 (+); no longer U501.9 (-)
- net SPKR_RIGHT_N: now also U501.5 (+); no longer U501.6 (-)
- net at C1.1, U501.14: now also U501.13 (-); no longer U501.12 (+)
- net at C1.1, U501.7: now also U501.6 (-); no longer U501.5 (+)
- net at C1.1, U501.8: now also U501.9 (-); no longer U501.10 (+)
Other:
- moved on the sheet: U501B, U501C, U501D, U502C
