File: connectors.kicad_sch (KiCad schematic)
At the start: 32 parts, among them J101 Power Terminal, J103 Mic 1 Connector, J104 Mic 2 Connector, J105 GPIO 0 Connector, J106 GPIO 1 Connector, J107 GPIO 2 Connector, J108 GPIO 3 Connector, J109 Speaker Right Connector, J110 Speaker Left Connector, J2 USB C Port

Commit message: ara ara
Parts:
- added J501: SWD Connector, Connector_PinSocket_1.00mm:PinSocket_1x04_P1.00mm_Vertical, symbol Connector:Conn_01x04_Pin
- added U503, U504, U505: ~, Diode_SMD:D_SOD-923, symbol Test:D5V0M1U2S9
Connections:
- net GND: now also J103.2 (Pin_2), J104.2 (Pin_2), J109.1 (Pin_1), J110.1 (Pin_1), U104.2, U105.2, U114.2, U115.2, U116.2, U117.2, J501.1 (Pin_1), U503.2, U504.2, U505.2
- net SPKR_LEFT_P_BUF: now also J110.3 (Pin_3); no longer J110.1 (Pin_1)
- net SPKR_RIGHT_P_BUF: now also J109.3 (Pin_3); no longer J109.1 (Pin_1)
- removed net GNDS: J103.2 (Pin_2), J104.2 (Pin_2), J109.3 (Pin_3), J110.3 (Pin_3), U104.2, U105.2, U114.2, U115.2, U116.2, U117.2
- new net MCU_SWCLK: J501.3 (Pin_3), U504.1
- new net MCU_SWDIO: J501.2 (Pin_2), U503.1
- new net RST: J501.4 (Pin_4), U505.1
