File: power.kicad_sch (KiCad schematic)
At the start: 5 parts, among them U401 TLV75733PDRV

Commit message: ara ara
Parts:
- removed R401, R402: 2.2k, Resistor_SMD:R_0402_1005Metric_Pad0.72x0.64mm_HandSolder, symbol Device:R_US
Changed lines of the file:
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@@
   (junction (at 144.78 91.44) (diameter 0) (color 0 0 0 0)
   )
-  (junction (at 40.64 99.06) (diameter 0) (color 0 0 0 0)
-  )
   (junction (at 130.81 104.14) (diameter 0) (color 0 0 0 0)
   )
@@
     (stroke (width 0) (type default))
   )
-  (wire (pts (xy 40.64 95.25) (xy 40.64 99.06))
-    (stroke (width 0) (type default))
-  )
   (wire (pts (xy 120.65 93.98) (xy 123.19 93.98))
     (stroke (width 0) (type default))
   )
-  (wire (pts (xy 40.64 83.82) (xy 40.64 87.63))
-    (stroke (width 0) (type default))
-  )
   (wire (pts (xy 144.78 104.14) (xy 144.78 99.06))
     (stroke (width 0) (type default))
   )
-  (wire (pts (xy 40.64 99.06) (xy 40.64 101.6))
-    (stroke (width 0) (type default))
-  )
   (wire (pts (xy 120.65 91.44) (xy 123.19 91.44))
     (stroke (width 0) (type default))
@@
     (stroke (width 0) (type default))
   )
-  (wire (pts (xy 40.64 99.06) (xy 44.45 99.06))
-    (stroke (width 0) (type default))
-  )
-  (wire (pts (xy 40.64 109.22) (xy 40.64 114.3))
-    (stroke (width 0) (type default))
-  )
   (wire (pts (xy 130.81 101.6) (xy 130.81 104.14))
     (stroke (width 0) (type default))
-  )
-  (symbol (lib_id "Device:R_US") (at 40.64 91.44 0) (unit 1)
-    (in_bom yes) (on_board yes) (dnp no) (fields_autoplaced)
-    (property "Reference" "R401" (at 43.18 90.17 0)
-      (effects (font (size 1.27 1.27)) (justify left))
-    )
-    (property "Value" "2.2k" (at 43.18 92.71 0)
-      (effects (font (size 1.27 1.27)) (justify left))
-    )
-    (property "Footprint" "Resistor_SMD:R_0402_1005Metric_Pad0.72x0.64mm_HandSolder" (at 41.656 91.694 90)
-      (effects (font (size 1.27 1.27)) hide)
-    )
-    (property "Datasheet" "~" (at 40.64 91.44 0)
-      (effects (font (size 1.27 1.27)) hide)
-    )
-    (pin "1")
-    (pin "2")
-    (instances
-      (project "AudioAmp"
-        (path "/7c40bb6d-39d1-4b91-a2f2-a85e74d3b158/54f4758a-8b57-4618-8682-2393a00ecf13"
-          (reference "R401") (unit 1)
-        )
-      )
-    )
   )
   (symbol (lib_id "Regulator_Linear:TLV75733PDRV") (at 130.81 93.98 0) (unit 1)
@@
     )
   )
-  (symbol (lib_id "Device:R_US") (at 40.64 105.41 0) (unit 1)
-    (in_bom yes) (on_board yes) (dnp no) (fields_autoplaced)
-    (property "Reference" "R402" (at 43.18 104.14 0)
-      (effects (font (size 1.27 1.27)) (justify left))
-    )
-    (property "Value" "2.2k" (at 43.18 106.68 0)
-      (effects (font (size 1.27 1.27)) (justify left))
-    )
-    (property "Footprint" "Resistor_SMD:R_0402_1005Metric_Pad0.72x0.64mm_HandSolder" (at 41.656 105.664 90)
-      (effects (font (size 1.27 1.27)) hide)
-    )
-    (property "Datasheet" "~" (at 40.64 105.41 0)
-      (effects (font (size 1.27 1.27)) hide)
-    )
-    (pin "1")
-    (pin "2")
-    (instances
-      (project "AudioAmp"
-        (path "/7c40bb6d-39d1-4b91-a2f2-a85e74d3b158/54f4758a-8b57-4618-8682-2393a00ecf13"
-          (reference "R402") (unit 1)
-        )
-      )
-    )
-  )
-  (symbol (lib_id "power:+5V") (at 40.64 83.82 0) (unit 1)
-    (in_bom yes) (on_board yes) (dnp no) (fields_autoplaced)
-    (property "Reference" "#PWR02" (at 40.64 87.63 0)
-      (effects (font (size 1.27 1.27)) hide)
-    )
-    (property "Value" "+5V" (at 40.64 78.74 0)
-      (effects (font (size 1.27 1.27)))
-    )
-    (property "Footprint" "" (at 40.64 83.82 0)
-      (effects (font (size 1.27 1.27)) hide)
-    )
-    (property "Datasheet" "" (at 40.64 83.82 0)
+  (symbol (lib_id "power:+5V") (at 107.95 86.36 0) (unit 1)
+    (in_bom yes) (on_board yes) (dnp no) (fields_autoplaced)
+    (property "Reference" "#PWR02" (at 107.95 90.17 0)
+      (effects (font (size 1.27 1.27)) hide)
+    )
+    (property "Value" "+5V" (at 107.95 81.28 0)
+      (effects (font (size 1.27 1.27)))
+    )
+    (property "Footprint" "" (at 107.95 86.36 0)
+      (effects (font (size 1.27 1.27)) hide)
+    )
+    (property "Datasheet" "" (at 107.95 86.36 0)
       (effects (font (size 1.27 1.27)) hide)
     )
@@
           (reference "#PWR02") (unit 1)
         )
-        (path "/7c40bb6d-39d1-4b91-a2f2-a85e74d3b158/d9f22c81-3656-48f7-9541-e4fbc6f14548"
-          (reference "#PWR024") (unit 1)
-        )
-        (path "/7c40bb6d-39d1-4b91-a2f2-a85e74d3b158/54f4758a-8b57-4618-8682-2393a00ecf13"
-          (reference "#PWR0401") (unit 1)
-        )
-      )
-    )
-  )
-  (symbol (lib_id "power:+5V") (at 107.95 86.36 0) (unit 1)
-    (in_bom yes) (on_board yes) (dnp no) (fields_autoplaced)
-    (property "Reference" "#PWR02" (at 107.95 90.17 0)
-      (effects (font (size 1.27 1.27)) hide)
-    )
-    (property "Value" "+5V" (at 107.95 81.28 0)
-      (effects (font (size 1.27 1.27)))
-    )
-    (property "Footprint" "" (at 107.95 86.36 0)
-      (effects (font (size 1.27 1.27)) hide)
-    )
-    (property "Datasheet" "" (at 107.95 86.36 0)
-      (effects (font (size 1.27 1.27)) hide)
-    )
-    (pin "1")
-    (instances
-      (project "AudioAmp"
-        (path "/7c40bb6d-39d1-4b91-a2f2-a85e74d3b158/97bd80ce-01ef-4bab-aca5-9a0417b7661d"
-          (reference "#PWR02") (unit 1)
-        )
         (path "/7c40bb6d-39d1-4b91-a2f2-a85e74d3b158/54f4758a-8b57-4618-8682-2393a00ecf13"
           (reference "#PWR0404") (unit 1)
@@
         )
       )
-    )
-  )
-  (symbol (lib_id "power:GND") (at 40.64 114.3 0) (unit 1)
-    (in_bom yes) (on_board yes) (dnp no) (fields_autoplaced)
-    (property "Reference" "#PWR011" (at 40.64 120.65 0)
-      (effects (font (size 1.27 1.27)) hide)
-    )
-    (property "Value" "GND" (at 40.64 119.38 0)
-      (effects (font (size 1.27 1.27)))
-    )
-    (property "Footprint" "" (at 40.64 114.3 0)
-      (effects (font (size 1.27 1.27)) hide)
-    )
-    (property "Datasheet" "" (at 40.64 114.3 0)
-      (effects (font (size 1.27 1.27)) hide)
-    )
-    (pin "1")
-    (instances
-      (project "AudioAmp"
-        (path "/7c40bb6d-39d1-4b91-a2f2-a85e74d3b158/97bd80ce-01ef-4bab-aca5-9a0417b7661d"
-          (reference "#PWR011") (unit 1)
-        )
-        (path "/7c40bb6d-39d1-4b91-a2f2-a85e74d3b158/54f4758a-8b57-4618-8682-2393a00ecf13"
-          (reference "#PWR0402") (unit 1)
-        )
-      )
-    )
-  )
-  (symbol (lib_id "power:GNDS") (at 44.45 99.06 90) (unit 1)
-    (in_bom yes) (on_board yes) (dnp no) (fields_autoplaced)
-    (property "Reference" "#PWR07" (at 50.8 99.06 0)
-      (effects (font (size 1.27 1.27)) hide)
-    )
-    (property "Value" "GNDS" (at 48.26 99.06 90)
-      (effects (font (size 1.27 1.27)) (justify right))
-    )
-    (property "Footprint" "" (at 44.45 99.06 0)
-      (effects (font (size 1.27 1.27)) hide)
-    )
-    (property "Datasheet" "" (at 44.45 99.06 0)
-      (effects (font (size 1.27 1.27)) hide)
-    )
-    (pin "1")
-    (instances
-      (project "AudioAmp"
-        (path "/7c40bb6d-39d1-4b91-a2f2-a85e74d3b158/97bd80ce-01ef-4bab-aca5-9a0417b7661d"
-          (reference "#PWR07") (unit 1)
-        )
-        (path "/7c40bb6d-39d1-4b91-a2f2-a85e74d3b158/54f4758a-8b57-4618-8682-2393a00ecf13"
-          (reference "#PWR0403") (unit 1)
-        )
-      )
